File: Circuits/Automatic_Piano/UART_to_USB.sch (KiCad schematic (older format))
At the start: 0 parts

Commit message: Completed MIDI to UART and UART to USB. Needs referencing
Parts:
- added C? (x2): 47pF, symbol Device:C_Small
- added C?: 10nF, symbol Device:C_Small
- added C? (x2): 100nF, symbol Device:C_Small
- added C?: 4.7uF, symbol Device:CP1_Small
- added FB?: MI0805K601R-10, Resistor_SMD:R_0805_2012Metric, symbol Device:Ferrite_Bead_Small
- added R? (x2): 280R, Resistor_SMD:R_0603_1608Metric, symbol Device:R_Small
- added U?: FT230XS, Package_SO:SSOP-16_3.9x4.9mm_P0.635mm, symbol Interface_USB:FT230XS
Connections:
- new net: FB?.1, U?.12 (VCC)
- new net: R?.2, U?.8 (USBDP)
- new net: C?.1, R?.2, U?.9 (USBDM)
- new net +3V3: C?.1, C?.1, C?.1
- new net 3V3_: C?.1, U?.10 (3V3OUT), U?.11 (~RESET), U?.3 (VCCIO)
- new net GND: C?.2, C?.2, C?.2, C?.2, C?.2, C?.2, U?.13 (GND), U?.5 (GND)
- new net UART_RX: U?.4 (RXD)
- new net UART_TX: U?.1 (TXD)
- new net USB_D+: C?.1, R?.1
- new net USB_D-: R?.1
- new net V_BUS: FB?.2
