File: Circuits/Automatic_Piano/CAN.sch (KiCad schematic (older format))
At the start: 0 parts

Commit message: Main Piano MIDI receiver completed. Might want indicator LEDS and more peripherals.
Parts:
- added C501: 100nF, symbol Device:C_Small
- added U501: SN65HVD232, Package_SO:SOIC-8_3.9x4.9mm_P1.27mm, symbol Interface_CAN_LIN:SN65HVD232
Connections:
- new net +3V3: C501.1, U501.3 (VCC)
- new net CAN_H: U501.7 (CANH)
- new net CAN_L: U501.6 (CANL)
- new net CAN_RX: U501.4 (R)
- new net CAN_TX: U501.1 (D)
- new net GND: C501.2, U501.2 (GND)
Changed lines of the file:
@@
 $Descr A4 11693 8268
 encoding utf-8
-Sheet 1 5
+Sheet 5 5
 Title ""
 Date ""
@@
 Comment4 ""
 $EndDescr
+$Comp
+L Interface_CAN_LIN:SN65HVD232 U501
+U 1 1 5E235FED
+P 5000 3250
+F 0 "U501" H 5150 3600 50  0000 C CNN
+F 1 "SN65HVD232" H 5350 3500 50  0000 C CNN
+F 2 "Package_SO:SOIC-8_3.9x4.9mm_P1.27mm" H 5000 2750 50  0001 C CNN
+F 3 "http://www.ti.com/lit/ds/symlink/sn65hvd230.pdf" H 4900 3650 50  0001 C CNN
+	1    5000 3250
+	1    0    0    -1
+$EndComp
+Text HLabel 4500 3150 0    50   Input ~ 0
+CAN_TX
+Text HLabel 4500 3250 0    50   Output ~ 0
+CAN_RX
+$Comp
+L power:+3.3V #PWR?
+U 1 1 5E23994C
+P 4500 2400
+AR Path="/5E18CB51/5E23994C" Ref="#PWR?"  Part="1"
+AR Path="/5E18D8EB/5E23994C" Ref="#PWR0501"  Part="1"
+F 0 "#PWR0501" H 4500 2250 50  0001 C CNN
+F 1 "+3.3V" H 4515 2573 50  0000 C CNN
+F 2 "" H 4500 2400 50  0001 C CNN
+F 3 "" H 4500 2400 50  0001 C CNN
+	1    4500 2400
+	1    0    0    -1
+$EndComp
+$Comp
+L power:GND #PWR?
+U 1 1 5E239952
+P 4500 2800
+AR Path="/5E18CB51/5E239952" Ref="#PWR?"  Part="1"
+AR Path="/5E18D8EB/5E239952" Ref="#PWR0502"  Part="1"
+F 0 "#PWR0502" H 4500 2550 50  0001 C CNN
+F 1 "GND" H 4505 2627 50  0000 C CNN
+F 2 "" H 4500 2800 50  0001 C CNN
+F 3 "" H 4500 2800 50  0001 C CNN
+	1    4500 2800
+	1    0    0    -1
+$EndComp
+Wire Wire Line
+	4500 2700 4500 2800
+$Comp
+L Device:C_Small C?
+U 1 1 5E239959
+P 4500 2600
+AR Path="/5E18D7E6/5E239959" Ref="C?"  Part="1"
+AR Path="/5E18CB51/5E239959" Ref="C?"  Part="1"
+AR Path="/5E18D8EB/5E239959" Ref="C501"  Part="1"
+F 0 "C501" H 4592 2646 50  0000 L CNN
+F 1 "100nF" H 4592 2555 50  0000 L CNN
+F 2 "" H 4500 2600 50  0001 C CNN
+F 3 "~" H 4500 2600 50  0001 C CNN
+	1    4500 2600
+	1    0    0    -1
+$EndComp
+Wire Wire Line
+	4500 2400 4500 2500
+Wire Wire Line
+	4500 3150 4600 3150
+Wire Wire Line
+	4500 3250 4600 3250
+$Comp
+L power:+3.3V #PWR?
+U 1 1 5E23A64A
+P 5000 2850
+AR Path="/5E18CB51/5E23A64A" Ref="#PWR?"  Part="1"
+AR Path="/5E18D8EB/5E23A64A" Ref="#PWR0503"  Part="1"
+F 0 "#PWR0503" H 5000 2700 50  0001 C CNN
+F 1 "+3.3V" H 5015 3023 50  0000 C CNN
+F 2 "" H 5000 2850 50  0001 C CNN
+F 3 "" H 5000 2850 50  0001 C CNN
+	1    5000 2850
+	1    0    0    -1
+$EndComp
+Wire Wire Line
+	5000 2950 5000 2850
+$Comp
+L power:GND #PWR?
+U 1 1 5E23ABAD
+P 5000 3750
+AR Path="/5E18CB51/5E23ABAD" Ref="#PWR?"  Part="1"
+AR Path="/5E18D8EB/5E23ABAD" Ref="#PWR0504"  Part="1"
+F 0 "#PWR0504" H 5000 3500 50  0001 C CNN
+F 1 "GND" H 5005 3577 50  0000 C CNN
+F 2 "" H 5000 3750 50  0001 C CNN
+F 3 "" H 5000 3750 50  0001 C CNN
+	1    5000 3750
+	1    0    0    -1
+$EndComp
+Wire Wire Line
+	5000 3650 5000 3750
+Wire Wire Line
+	5400 3250 5500 3250
+Wire Wire Line
+	5400 3350 5500 3350
+Text HLabel 5500 3250 2    50   Output ~ 0
+CAN_H
+Text HLabel 5500 3350 2    50   Output ~ 0
+CAN_L
 $EndSCHEMATC
